File: samd21pad.kicad_pcb (KiCad board)
At the start: 2 copper layers, 119.3 x 119.3 mm, 49 parts, among them J1 USB_C_Receptacle_USB2.0, J2 Conn_ARM_SWD_TagConnect_TC203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, SW1 SW_Push, SW10 SKQGAKE020, SW2 SW_Push, SW3 SW_Push, SW4 SW_Push, SW5 SW_Push, SW6 SW_Push, SW7 SW_Push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

Commit message: Fix the solder nut part/JLC number.
Parts:
- H1, H2, H3, H4: value SMTSO2030 -> SMTSO2040
Changed lines of the file:
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@@
     (descr "Mounting Hole 3mm")
     (tags "mounting hole 3mm")
-    (property "LCSC Part Number" "C2928170")
+    (property "LCSC Part Number" "C2916349 ")
     (property "MPN" "")
     (property "Sheetfile" "samd21pad.kicad_sch")
@@
         (effects (font (size 1 1) (thickness 0.15)) (justify mirror))
     )
-    (fp_text value "SMTSO2030" (at 0 -4) (layer "B.Fab")
+    (fp_text value "SMTSO2040" (at 0 -4) (layer "B.Fab")
         (effects (font (size 1 1) (thickness 0.15)) (justify mirror))
     )
@@
     (descr "Mounting Hole 3mm")
     (tags "mounting hole 3mm")
-    (property "LCSC Part Number" "C2928170")
+    (property "LCSC Part Number" "C2916349")
     (property "MPN" "")
     (property "Sheetfile" "samd21pad.kicad_sch")
@@
         (effects (font (size 1 1) (thickness 0.15)) (justify mirror))
     )
-    (fp_text value "SMTSO2030" (at 0 -4) (layer "B.Fab")
+    (fp_text value "SMTSO2040" (at 0 -4) (layer "B.Fab")
         (effects (font (size 1 1) (thickness 0.15)) (justify mirror))
     )
@@
     (descr "Mounting Hole 3mm")
     (tags "mounting hole 3mm")
-    (property "LCSC Part Number" "C2928170")
+    (property "LCSC Part Number" "C2916349")
     (property "MPN" "")
     (property "Sheetfile" "samd21pad.kicad_sch")
@@
         (effects (font (size 1 1) (thickness 0.15)) (justify mirror))
     )
-    (fp_text value "SMTSO2030" (at 0 -4) (layer "B.Fab")
+    (fp_text value "SMTSO2040" (at 0 -4) (layer "B.Fab")
         (effects (font (size 1 1) (thickness 0.15)) (justify mirror))
     )
@@
     (descr "SOT, 5 Pin (https://www.jedec.org/sites/default/files/docs/Mo-178c.PDF variant AA), generated with kicad-footprint-generator ipc_gullwing_generator.py")
     (tags "SOT TO_SOT_SMD")
-    (property "LCSC Part Number" "C51118")
+    (property "LCSC Part Number" "C3021085")
     (property "MPN" "AP2112K-3.3")
     (property "Sheetfile" "samd21pad.kicad_sch")
@@
     (descr "Mounting Hole 3mm")
     (tags "mounting hole 3mm")
-    (property "LCSC Part Number" "C2928170")
+    (property "LCSC Part Number" "C2916349")
     (property "MPN" "")
     (property "Sheetfile" "samd21pad.kicad_sch")
@@
         (effects (font (size 1 1) (thickness 0.15)) (justify mirror))
     )
-    (fp_text value "SMTSO2030" (at 0 -4) (layer "B.Fab")
-        (effects (font (size 1 1) (thickness 0.15)) (justify mirror))
-    )
+    (fp_text value "SMTSO2040" (at 0 -4) (layer "B.Fab")
+        (effects (font (size 1 1) (thickness 0.15)) (justify mirror))
+    )

Commit message: Tweaks for USB shield handling, nuke meetup silk.
Parts:
- removed C4: 4.5nF, Capacitor_SMD:C_0805_2012Metric
- removed G***: LOGO, samd21pad:smk-logo-40x40
- removed R4: 1M, Resistor_SMD:R_0805_2012Metric
Connections:
- J1 pad S1: Net-(J1-SHIELD) -> GND
Routing:
- net Net-(J1-SHIELD): track 21.6 -> 0.00 mm
- net GND: track 39.4 -> 55.6 mm
Other:
- board text removed: "2023.07.29"
